Commit message: Connect G1 to the TB4 base_link

File: manipulation/nav2_minimal_tb4_description/urdf/standard/turtlebot4.urdf.xacro (robot description, xacro)
@@ -1,4 +1,5 @@
 <?xml version="1.0" ?>
 <robot name="turtlebot4" xmlns:xacro="http://ros.org/wiki/xacro">
+<xacro:include filename="$(find nartech_ros)/g1_description/urdf/g1_macro.urdf.xacro" />
 <!--
 <gazebo>
@@ -72,4 +73,5 @@
   <!-- Turtlebot4 shell definition -->
   <link name="shell_link">
+    <!-- Hide the visual for now
     <visual>
       <origin xyz="0 0 0" rpy="${pi/2} 0 ${pi/2}"/>
@@ -77,5 +79,5 @@
         <mesh filename="package://nav2_minimal_tb4_description/meshes/shell.dae" scale="1 1 1" />
       </geometry>
-    </visual>
+    </visual> -->
     <collision name="shell_collision">
       <geometry>
@@ -143,3 +145,9 @@
     use_sim="$(arg use_sim)"
     use_fake_hardware="$(arg use_fake_hardware)" />
+  <!-- Attach Unitree G1 as a payload on the TB4 base_link.
+       Adjust xyz to position the G1 pelvis above the base.
+       For example, 0.0, 0.0, 0.25m above the base_link. -->
+  <xacro:g1_attach parent_link="base_link"
+                   xyz="0 0 0.25"
+                   rpy="0 0 0" />
 </robot>
